Commit message: 1.0.6

File: roch/roch_description/urdf/roch.urdf.xacro (robot description, xacro)
@@ -101,7 +101,7 @@
       </inertial>
    </link>
-<!--                 modify                           -->
-<!--              range_z: -0.007 ~ -0.008                              -->
-<!--                                            -->
+<!--                 modify                     -->
+<!--              range_z: -0.007 ~ -0.008      -->
+<!--        if not modify in gazebo will shack  -->
 <!--                                            -->
 <!--                                            -->

File: roch/roch_description/urdf/roch_library.urdf.xacro (robot description, xacro)
@@ -16,4 +16,7 @@
   <xacro:include filename="$(find roch_description)/urdf/sensors/asus_xtion_pro_offset.urdf.xacro"/>
   <xacro:include filename="$(find roch_description)/urdf/sensors/kinect_camera.urdf.xacro"/>
+  <xacro:include filename="$(find roch_description)/urdf/sensors/r200.urdf.xacro"/>
+  <!-- 2D Laser -->
   <xacro:include filename="$(find roch_description)/urdf/sensors/ls_ls01c.urdf.xacro"/>
+  <xacro:include filename="$(find roch_description)/urdf/sensors/rplidar.urdf.xacro"/>
 </robot>

File: roch/roch_description/urdf/roch_properties.urdf.xacro (robot description, xacro)
@@ -19,15 +19,24 @@
      (currently in development and awaiting feedback)
    -->
-	<property name="asus_xtion_px" value="-0.145" />
-	<property name="asus_xtion_py" value="-0.025" />
-	<property name="asus_xtion_pz" value="0.721" />
-	<property name="asus_xtion_or" value="0" />
-	<property name="asus_xtion_op" value="0" />
-	<property name="asus_xtion_oy" value="0" />
-	<property name="kinect_px" value="-0.145" />
-	<property name="kinect_py" value="-0.025" />
-	<property name="kinect_pz" value="0.721" />
-	<property name="kinect_or" value="0" />
-	<property name="kinect_op" value="0" />
-	<property name="kinect_oy" value="0" />
+<!-- asus xtion param -->
+  <property name="asus_xtion_px" value="-0.145" />
+  <property name="asus_xtion_py" value="-0.025" />
+  <property name="asus_xtion_pz" value="0.721" />
+  <property name="asus_xtion_or" value="0" />
+  <property name="asus_xtion_op" value="0" />
+  <property name="asus_xtion_oy" value="0" />
+<!-- kinect param -->
+  <property name="kinect_px" value="-0.145" />
+  <property name="kinect_py" value="-0.025" />
+  <property name="kinect_pz" value="0.721" />
+  <property name="kinect_or" value="0" />
+  <property name="kinect_op" value="0" />
+  <property name="kinect_oy" value="0" />
+<!-- Intel R200 param -->
+  <property name="r200_px" value="-0.135" />
+  <property name="r200_py" value="-0.065" />
+  <property name="r200_pz" value="0.7" />
+  <property name="r200_or" value="0" />
+  <property name="r200_op" value="0" />
+  <property name="r200_oy" value="0" />
 </robot>

File: roch/roch_description/urdf/sensors/ls_ls01c.urdf.xacro (robot description, xacro)
@@ -60,5 +60,5 @@
     <link name="base_laser"/>
     <joint name="base_laser_joint" type="fixed">
-      <origin xyz="0 0 0" rpy=" 0 ${M_PI} 0" />
+      <origin xyz="0 0 0.04076" rpy=" ${M_PI} 0 0" />
       <parent link="base_laser_link" />
       <child link="base_laser" />
